Commit message: move bot script added

File: ros/bot/vishwajeet/ethan_description/urdf/ethan.xacro (robot description, xacro)
@@ -34,13 +34,7 @@
     </inertial>
   </xacro:macro>
-   <link name="base_footprint"/>
-  <joint name="base_joint" type="fixed">
-    <parent link="base_footprint"/>
-    <child link="link_chassis"/>
-    <origin xyz="0.0 0.0 0.010" rpy="0 0 0"/>
-  </joint>
   <link name="link_chassis">
    <!-- pose and inertial -->
-   <!-- <pose>0 0 0.5 0 0 0</pose> -->
+   <pose>0 0 0.5 0 0 0</pose>
    <inertial>
     <mass value="${mass}" />
@@ -64,8 +58,8 @@
 <xacro:link_wheel name="link_right_wheel_back" mass="${wheel_mass}" r="${wheel_radius}" l="${wheel_length}" />
 <xacro:link_wheel name="link_left_wheel_back" mass="${wheel_mass}" r="${wheel_radius}" l="${wheel_length}"/>
-<xacro:joint_wheel name="joint_right_wheel_front"  child="link_right_wheel_front"  origin_xyz="0.17 -0.195 -0.0525"  />
-<xacro:joint_wheel name="joint_left_wheel_front"   child="link_left_wheel_front"   origin_xyz="0.17 0.195 -0.0525"  />
-<xacro:joint_wheel name="joint_right_wheel_back"  child="link_right_wheel_back"  origin_xyz="-0.17 -0.195 -0.0525"  />
-<xacro:joint_wheel name="joint_left_wheel_back"   child="link_left_wheel_back"   origin_xyz="-0.17 0.195 -0.0525"  />
+<xacro:joint_wheel name="joint_right_wheel_front"  child="link_right_wheel_front"  origin_xyz="0.17 0.195 -0.0525"  />
+<xacro:joint_wheel name="joint_left_wheel_front"   child="link_left_wheel_front"   origin_xyz="0.17 -0.195 -0.0525"  />
+<xacro:joint_wheel name="joint_right_wheel_back"  child="link_right_wheel_back"  origin_xyz="-0.17 0.195 -0.0525"  />
+<xacro:joint_wheel name="joint_left_wheel_back"   child="link_left_wheel_back"   origin_xyz="-0.17 -0.195 -0.0525"  />
 <!-- <xacro:transmission trans="link_left_wheel_front_trans" motor="link_left_wheel_front_motor" joint="joint_left_wheel_front"  /> -->
 <link name="left_scissor_hinge_front">
@@ -469,5 +463,5 @@
     <odometryTopic>odom</odometryTopic>
     <odometryFrame>odom</odometryFrame>
-    <robotBaseFrame>base_footprint</robotBaseFrame>
+    <robotBaseFrame>link_chassis</robotBaseFrame>
   </plugin>
 </gazebo>

File: ros/bot/vishwajeet/ethan_description/urdf/gazebo.xacro (robot description, xacro)
@@ -49,48 +49,77 @@
   <!-- camera -->
   <gazebo reference="camera_link">
-    <sensor type="depth" name="realsense_R200">
-      <always_on>true</always_on>
+  <sensor name="camera_link_camera" type="depth">
+    <update_rate>20</update_rate>
+    <camera>
+      <horizontal_fov>1.047198</horizontal_fov>
+      <image>
+        <width>640</width>
+        <height>480</height>
+        <format>R8G8B8</format>
+      </image>
+      <clip>
+        <near>0.05</near>
+        <far>3</far>
+      </clip>
+    </camera>
+    <plugin name="camera_link_controller" filename="libgazebo_ros_openni_kinect.so">
+      <baseline>0.2</baseline>
+      <alwaysOn>true</alwaysOn>
+      <updateRate>1.0</updateRate>
+      <cameraName>camera</cameraName>
+      <imageTopicName>camera/color/image_raw</imageTopicName>
+      <cameraInfoTopicName>/camera/color/camera_info</cameraInfoTopicName>
+      <depthImageTopicName>/camera/depth/image_raw</depthImageTopicName>
+      <depthImageInfoTopicName>/camera/depth/camera_info</depthImageInfoTopicName>
+      <pointCloudTopicName>/camera/depth/points</pointCloudTopicName>
+      <frameName>camera_frame</frameName>
+      <pointCloudCutoff>0.5</pointCloudCutoff>
+      <pointCloudCutoffMax>3.0</pointCloudCutoffMax>
+      <distortionK1>0.00000001</distortionK1>
+      <distortionK2>0.00000001</distortionK2>
+      <distortionK3>0.00000001</distortionK3>
+      <distortionT1>0.00000001</distortionT1>
+      <distortionT2>0.00000001</distortionT2>
+      <CxPrime>0</CxPrime>
+      <Cx>0</Cx>
+      <Cy>0</Cy>
+      <focalLength>0</focalLength>
+      <hackBaseline>0</hackBaseline>
+    </plugin>
+  </sensor>
+</gazebo>
+ <!-- hokuyo -->
+<!--   <gazebo reference="hokuyo_link">
+    <sensor type="gpu_ray" name="head_hokuyo_sensor">
+      <pose>0 0 0 0 0 0</pose>
       <visualize>false</visualize>
-      <camera>
-          <horizontal_fov>1.3439</horizontal_fov>
-          <image>
-              <width>1920</width>
-              <height>1080</height>
-              <format>R8G8B8</format>
-          </image>
-          <depth_camera></depth_camera>
-          <clip>
-              <near>0.03</near>
-              <far>100</far>
-          </clip>
-      </camera>
-      <plugin name="camera_controller" filename="libgazebo_ros_openni_kinect.so">
-        <baseline>0.2</baseline>
-        <alwaysOn>true</alwaysOn>
-        <updateRate>30.0</updateRate>
-        <cameraName>camera</cameraName>
-        <frameName>camera_rgb_optical_frame</frameName>
-        <imageTopicName>rgb/image_raw</imageTopicName>
-        <depthImageTopicName>depth/image_raw</depthImageTopicName>
-        <pointCloudTopicName>depth/points</pointCloudTopicName>
-        <cameraInfoTopicName>rgb/camera_info</cameraInfoTopicName>
-        <depthImageCameraInfoTopicName>depth/camera_info</depthImageCameraInfoTopicName>
-        <pointCloudCutoff>0.4</pointCloudCutoff>
-            <hackBaseline>0.07</hackBaseline>
-            <distortionK1>0.0</distortionK1>
-            <distortionK2>0.0</distortionK2>
-            <distortionK3>0.0</distortionK3>
-            <distortionT1>0.0</distortionT1>
-            <distortionT2>0.0</distortionT2>
-        <CxPrime>0.0</CxPrime>
-        <Cx>0.0</Cx>
-        <Cy>0.0</Cy>
-        <focalLength>0</focalLength>
-        <hackBaseline>0</hackBaseline>
+      <update_rate>40</update_rate>
+      <ray>
+        <scan>
+          <horizontal>
+            <samples>720</samples>
+            <resolution>1</resolution>
+            <min_angle>-3.14159</min_angle>
+            <max_angle>3.14159</max_angle>
+          </horizontal>
+        </scan>
+        <range>
+          <min>0.10</min>
+          <max>30.0</max>
+          <resolution>0.01</resolution>
+        </range>
+        <noise>
+          <type>gaussian</type>
+          <mean>0.0</mean>
+          <stddev>0.01</stddev>
+        </noise>
+      </ray>
+      <plugin name="gazebo_ros_head_hokuyo_controller" filename="libgazebo_ros_gpu_laser.so">
+        <topicName>/scan</topicName>
+        <frameName>hokuyo_link</frameName>
       </plugin>
     </sensor>
-  </gazebo>
- <!-- hokuyo -->
-   <gazebo reference="hokuyo_link">
+  </gazebo> -->
+    <gazebo reference="hokuyo_link">
     <material>Gazebo/FlatBlack</material>
     <sensor type="ray" name="lds_lfcd_sensor">
@@ -120,5 +149,5 @@
       <plugin name="gazebo_ros_lds_lfcd_controller" filename="libgazebo_ros_laser.so">
         <topicName>scan</topicName>
-        <frameName>base_scan</frameName>
+        <frameName>hokuyo_link</frameName>
       </plugin>
     </sensor>

Commit message: changes in laser

File: ros/bot/vishwajeet/ethan_description/urdf/ethan.xacro (robot description, xacro)
@@ -46,11 +46,9 @@
     </geometry>
   </collision>
-  <visual>
-    <origin rpy="0 0 0" xyz="0 0 0"/>
+  <visual name="visual_chassis">
     <geometry>
       <box size="${length} ${width} ${height}"/>
     </geometry>
-    <material name="blue"/>
-  </visual>
+  </visual>>
 </link>
 <xacro:link_wheel name="link_right_wheel_front" mass="${wheel_mass}" r="${wheel_radius}" l="${wheel_length}" />

File: ros/bot/vishwajeet/ethan_description/urdf/gazebo.xacro (robot description, xacro)
@@ -90,9 +90,9 @@
 </gazebo>
  <!-- hokuyo -->
-<!--   <gazebo reference="hokuyo_link">
-    <sensor type="gpu_ray" name="head_hokuyo_sensor">
+  <gazebo reference="hokuyo_link">
+    <sensor type="ray" name="head_hokuyo_sensor">
       <pose>0 0 0 0 0 0</pose>
-      <visualize>false</visualize>
-      <update_rate>40</update_rate>
+      <visualize>true</visualize>
+      <update_rate>20</update_rate>
       <ray>
         <scan>
@@ -100,11 +100,11 @@
             <samples>720</samples>
             <resolution>1</resolution>
-            <min_angle>-3.14159</min_angle>
-            <max_angle>3.14159</max_angle>
+            <min_angle>-1.570796</min_angle>
+            <max_angle>1.570796</max_angle>
           </horizontal>
         </scan>
         <range>
           <min>0.10</min>
-          <max>30.0</max>
+          <max>10.0</max>
           <resolution>0.01</resolution>
         </range>
@@ -115,11 +115,11 @@
         </noise>
       </ray>
-      <plugin name="gazebo_ros_head_hokuyo_controller" filename="libgazebo_ros_gpu_laser.so">
+      <plugin name="gazebo_ros_head_hokuyo_controller" filename="libgazebo_ros_laser.so">
         <topicName>/scan</topicName>
-        <frameName>hokuyo_link</frameName>
+        <frameName>sensor_laser</frameName>
       </plugin>
     </sensor>
-  </gazebo> -->
-    <gazebo reference="hokuyo_link">
+  </gazebo>
+<!--     <gazebo reference="hokuyo_link">
     <material>Gazebo/FlatBlack</material>
     <sensor type="ray" name="lds_lfcd_sensor">
@@ -152,5 +152,5 @@
       </plugin>
     </sensor>
-  </gazebo>
+  </gazebo> -->
   <!--
     Now we are ready to add control to our robot. We will add a new element called plugin to our xacro file. We will add a differential drive plugin to our robot. The new tag looks like follows:

Commit message: bot updated

File: ros/bot/vishwajeet/ethan_description/urdf/ethan.xacro (robot description, xacro)
@@ -342,6 +342,6 @@
 <joint name="hokuyo_joint" type="fixed">
   <axis xyz="0 1 0" />
-  <origin xyz="-0.02 0 0.09" rpy="0 0 0"/>
-  <parent link="upper_platform"/>
+  <origin xyz="0.21 0 0.09" rpy="0 0 0"/>
+  <parent link="link_chassis"/>
   <child link="hokuyo_link"/>
 </joint>

File: ros/bot/vishwajeet/ethan_description/urdf/gazebo.xacro (robot description, xacro)
@@ -117,5 +117,5 @@
       <plugin name="gazebo_ros_head_hokuyo_controller" filename="libgazebo_ros_laser.so">
         <topicName>/scan</topicName>
-        <frameName>sensor_laser</frameName>
+        <frameName>hokuyo_link</frameName>
       </plugin>
     </sensor>

Commit message: package updated

File: ros/bot/vishwajeet/ethan_description/urdf/ethan.xacro (robot description, xacro)
@@ -6,5 +6,5 @@
   <xacro:property name="width" value="0.4" />
   <xacro:property name="height" value="0.005" />
-  <xacro:property name="arm_l" value="0.1" />
+  <xacro:property name="arm_l" value="0.13" />
   <xacro:property name="arm_r" value="0.01" />
   <xacro:property name="arm2_mass" value="0.2" />
@@ -18,5 +18,5 @@
   <xacro:property name="holder_r" value="0.01" />
   <xacro:property name="holder_mass" value="0.2" />
-  <xacro:property name="mass" value="50" />
+  <xacro:property name="mass" value="100" />
   <xacro:property name="hinge_r" value="0.02" />
   <xacro:property name="hinge_l" value="0.01" />
@@ -24,5 +24,5 @@
   <xacro:include filename="$(find ethan_description)/urdf/macro.xacro" />
   <xacro:include filename="$(find ethan_description)/urdf/gazebo.xacro" />
-  <xacro:property name="wheel_mass" value="2" />
+  <xacro:property name="wheel_mass" value="10" />
   <xacro:property name="wheel_radius" value="0.05" />
   <xacro:property name="wheel_length" value="0.03" />
@@ -61,4 +61,5 @@
 <xacro:joint_wheel name="joint_left_wheel_back"   child="link_left_wheel_back"   origin_xyz="-0.17 -0.195 -0.0525"  />
 <!-- <xacro:transmission trans="link_left_wheel_front_trans" motor="link_left_wheel_front_motor" joint="joint_left_wheel_front"  /> -->
+<!--
 <link name="left_scissor_hinge_front">
   <inertial>
@@ -162,5 +163,5 @@
   <axis xyz="1 0 0" />
   <limit effort="10000" lower="0.0" upper="0.15" velocity="1" />
-</joint>
+</joint> -->
 <link name="upper_platform">
   <inertial>

File: ros/bot/vishwajeet/ethan_description/urdf/gazebo.xacro (robot description, xacro)
@@ -74,5 +74,5 @@
       <pointCloudTopicName>/camera/depth/points</pointCloudTopicName>
       <frameName>camera_frame</frameName>
-      <pointCloudCutoff>0.5</pointCloudCutoff>
+      <pointCloudCutoff>0.1</pointCloudCutoff>
       <pointCloudCutoffMax>3.0</pointCloudCutoffMax>
       <distortionK1>0.00000001</distortionK1>

Commit message: updated

File: ros/bot/vishwajeet/ethan_description/urdf/ethan.xacro (robot description, xacro)
@@ -18,5 +18,5 @@
   <xacro:property name="holder_r" value="0.01" />
   <xacro:property name="holder_mass" value="0.2" />
-  <xacro:property name="mass" value="100" />
+  <xacro:property name="mass" value="80" />
   <xacro:property name="hinge_r" value="0.02" />
   <xacro:property name="hinge_l" value="0.01" />
@@ -24,5 +24,5 @@
   <xacro:include filename="$(find ethan_description)/urdf/macro.xacro" />
   <xacro:include filename="$(find ethan_description)/urdf/gazebo.xacro" />
-  <xacro:property name="wheel_mass" value="10" />
+  <xacro:property name="wheel_mass" value="5" />
   <xacro:property name="wheel_radius" value="0.05" />
   <xacro:property name="wheel_length" value="0.03" />

File: ros/bot/vishwajeet/ethan_description/urdf/gazebo.xacro (robot description, xacro)
@@ -48,50 +48,52 @@
   </gazebo>
   <!-- camera -->
-  <gazebo reference="camera_link">
-  <sensor name="camera_link_camera" type="depth">
-    <update_rate>20</update_rate>
-    <camera>
-      <horizontal_fov>1.047198</horizontal_fov>
-      <image>
-        <width>640</width>
-        <height>480</height>
-        <format>R8G8B8</format>
-      </image>
-      <clip>
-        <near>0.05</near>
-        <far>3</far>
-      </clip>
-    </camera>
-    <plugin name="camera_link_controller" filename="libgazebo_ros_openni_kinect.so">
-      <baseline>0.2</baseline>
-      <alwaysOn>true</alwaysOn>
-      <updateRate>1.0</updateRate>
-      <cameraName>camera</cameraName>
-      <imageTopicName>camera/color/image_raw</imageTopicName>
-      <cameraInfoTopicName>/camera/color/camera_info</cameraInfoTopicName>
-      <depthImageTopicName>/camera/depth/image_raw</depthImageTopicName>
-      <depthImageInfoTopicName>/camera/depth/camera_info</depthImageInfoTopicName>
-      <pointCloudTopicName>/camera/depth/points</pointCloudTopicName>
-      <frameName>camera_frame</frameName>
-      <pointCloudCutoff>0.1</pointCloudCutoff>
-      <pointCloudCutoffMax>3.0</pointCloudCutoffMax>
-      <distortionK1>0.00000001</distortionK1>
-      <distortionK2>0.00000001</distortionK2>
-      <distortionK3>0.00000001</distortionK3>
-      <distortionT1>0.00000001</distortionT1>
-      <distortionT2>0.00000001</distortionT2>
-      <CxPrime>0</CxPrime>
-      <Cx>0</Cx>
-      <Cy>0</Cy>
-      <focalLength>0</focalLength>
-      <hackBaseline>0</hackBaseline>
-    </plugin>
-  </sensor>
-</gazebo>
+    <gazebo reference="camera_link">
+    <sensor type="depth" name="realsense_R200">
+      <always_on>true</always_on>
+      <visualize>false</visualize>
+      <camera>
+          <horizontal_fov>1.3439</horizontal_fov>
+          <image>
+              <width>1920</width>
+              <height>1080</height>
+              <format>R8G8B8</format>
+          </image>
+          <depth_camera></depth_camera>
+          <clip>
+              <near>0.03</near>
+              <far>100</far>
+          </clip>
+      </camera>
+      <plugin name="camera_controller" filename="libgazebo_ros_openni_kinect.so">
+        <baseline>0.2</baseline>
+        <alwaysOn>true</alwaysOn>
+        <updateRate>30.0</updateRate>
+        <cameraName>camera</cameraName>
+        <frameName>camera_rgb_optical_frame</frameName>
+        <imageTopicName>rgb/image_raw</imageTopicName>
+        <depthImageTopicName>depth/image_raw</depthImageTopicName>
+        <pointCloudTopicName>depth/points</pointCloudTopicName>
+        <cameraInfoTopicName>rgb/camera_info</cameraInfoTopicName>
+        <depthImageCameraInfoTopicName>depth/camera_info</depthImageCameraInfoTopicName>
+        <pointCloudCutoff>0.1</pointCloudCutoff>
+            <hackBaseline>0.01</hackBaseline>
+            <distortionK1>0.0</distortionK1>
+            <distortionK2>0.0</distortionK2>
+            <distortionK3>0.0</distortionK3>
+            <distortionT1>0.0</distortionT1>
+            <distortionT2>0.0</distortionT2>
+        <CxPrime>0.0</CxPrime>
+        <Cx>0.0</Cx>
+        <Cy>0.0</Cy>
+        <focalLength>0</focalLength>
+        <hackBaseline>0</hackBaseline>
+      </plugin>
+    </sensor>
+  </gazebo>
  <!-- hokuyo -->
   <gazebo reference="hokuyo_link">
     <sensor type="ray" name="head_hokuyo_sensor">
       <pose>0 0 0 0 0 0</pose>
-      <visualize>true</visualize>
+      <!-- <visualize>true</visualize> -->
       <update_rate>20</update_rate>
       <ray>
